File: td-deflect/power_supply.kicad_sch (KiCad schematic)
At the start: 68 parts, among them J13 Conn_01x02_Male, J14 Conn_01x02_Male, J15 Conn_01x02_Male, J18 Conn_01x02_Male, J2 Conn_01x02_Male, J8 Conn_01x02_Male, J9 Conn_01x02_Male, Q12 C2M0045170D, Q13 BSC082N10LSG, U13 MCP1416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

Commit message: Implemented some of the ToDos
Replaced current transformer for horizontal current measurement with a shunt  Replaced R22 with a bigger resistor (0.5W)  Replaced SiC-MOSFETs with smaller and cheaper alternatives  Removed HOT_CURRENT measurement  Replaced Q1 & Q3 with BSC600
Parts:
- Q12: value C2M0045170D -> LSIC1MO170E0750; Digikey C2M0045170D-ND -> 18-LSIC1MO170E0750-ND
