File: td-deflect/uc.kicad_sch (KiCad schematic)
At the start: 18 parts, among them J4 Conn_ARM_JTAG_SWD_10, J6 Conn_01x06_Male, U12 LM1117-5.0, U2 STM32F722RETx, U3 INA193, U4 TPS70933, X1 SG-8002CA

Commit message: Implemented some of the ToDos
Replaced current transformer for horizontal current measurement with a shunt  Replaced R22 with a bigger resistor (0.5W)  Replaced SiC-MOSFETs with smaller and cheaper alternatives  Removed HOT_CURRENT measurement  Replaced Q1 & Q3 with BSC600
Parts:
- removed U3: INA193, Package_TO_SOT_SMD:SOT-23-5, symbol Amplifier_Current:INA193
Connections:
- net hot_current_adc: no longer names the net of U2.15 (PA1)
- no-connect marks 26 -> 27
Other:
- note removed: "todo: drop this current sense, it's useless"
